File: link.sch (KiCad schematic (older format))
At the start: 34 parts, among them J1 Link, J2 Standard, J3 USB_C_Receptacle_USB2.0, J4 Conn_01x08, J5 Conn_01x08, Q1 MMBT3904, Q2 MMBT3904, U1 CP2104

Commit message: Release revC
Parts:
- removed D1: SP0504BAHT, Package_TO_SOT_SMD:SOT-23-5, symbol Power_Protection:SP0504BAHT
- removed JP1: NC, Jumper:SolderJumper-2_P1.3mm_Open_TrianglePad1.0x1.5mm, symbol Device:Jumper_NC_Small
- removed Q1, Q2: MMBT3904, Package_TO_SOT_SMD:SOT-23, symbol Transistor_BJT:MMBT3904
- removed U1: CP2104, Package_DFN_QFN:QFN-24-1EP_4x4mm_P0.5mm_EP2.6x2.6mm, symbol Interface_USB:CP2104
- added C6: 1uF, Capacitor_SMD:C_0603_1608Metric, symbol Device:C
- added D1: SP0503BAHT, Package_TO_SOT_SMD:SOT-143, symbol Power_Protection:SP0503BAHT
- added Q1: UMH3N, Package_TO_SOT_SMD:SOT-363_SC-70-6, symbol Transistor_BJT:UMH3N
- added U1: CP2102N-A01-GQFN28, Package_DFN_QFN:QFN-28-1EP_5x5mm_P0.5mm_EP3.35x3.35mm, symbol Interface_USB:CP2102N-A01-GQFN28
- added U2: LR1107, Package_TO_SOT_SMD:SOT-89-3, symbol voltlog:LR1107
- C1: footprint Capacitor_SMD:C_0603_1608Metric -> Capacitor_SMD:C_1206_3216Metric
- J3: footprint Voltlog:TYPE-C-31-M-12 -> voltlog:TYPE-C-31-M-12
- R1: footprint Resistor_SMD:R_0603_1608Metric -> Resistor_SMD:R_1206_3216Metric
- R6: value 10K -> 1K
- R7: value 10K -> 22.1K
- R8: value 10K -> 47.5K
Connections:
- net 3.45V is gone; now on net +3V3: C3.1, C4.1, D2.2 (A), D3.2 (A), J1.6 (Pin_6), J2.6 (Pin_6), J4.7 (Pin_7)
- net VIO is gone; now on net ~RST: J4.2 (Pin_2), R6.2
- net CTS: now also U1.23 (~CTS)
- net DCD: now also U1.1 (~DCD)
- net DM: now also D1.4 (K), U1.5 (D-)
- net DP: now also D1.3 (K), U1.4 (D+)
- net DSR: now also U1.27 (~DSR)
- net DTR: now also Q1.1 (E1), Q1.5 (B2), U1.28 (~DTR); no longer R7.2
- net EN: now also C6.1, Q1.3 (C2)
- net GND: now also R8.2, C6.2, D1.1 (A), U1.29 (GND), U1.3 (GND), U2.1 (GND); no longer J4.3 (Pin_3)
- net GPIO0: now also R4.2, U1.19 (~TXT~/GPIO.0); no longer R5.2
- net GPIO1: now also R5.2, U1.18 (~RXT~/GPIO.1); no longer R4.2
- net GPIO2: now also U1.17 (RS485/GPIO.2)
- net GPIO3: now also U1.16 (~WAKEUP~/GPIO.3)
- net IO0: now also Q1.6 (C1)
- net RI: now also U1.2 (~RI~/CLK)
- net RTS: now also Q1.2 (B1), Q1.4 (E2), U1.24 (~RTS); no longer R8.2
- net RXD: now also U1.25 (RXD)
- net SUSPEND: now also J4.4 (Pin_4), U1.12 (SUSPEND); no longer J5.7 (Pin_7)
- net TXD: now also U1.26 (TXD)
- net USB_PWR: now also D1.2 (K)
- net VBUS: now also R7.1, U2.2 (VIN)
- net ~RST: now also U1.9 (~RSTb); no longer J4.4 (Pin_4), R6.1
- net ~SUSPEND: now also J4.3 (Pin_3), U1.11 (~SUSPENDb); no longer J5.8 (Pin_8)
- net +3V3: now reaches C5.1
- net +3V3: now also R6.1, U1.6 (VDD), U1.7 (REGIN), U2.3 (VOUT)
- net at R8.1: now also R7.2, U1.8 (VBUS)
- new net CHR0: U1.15 (CHR0)
- new net CHR1: U1.14 (CHR1)
- new net CHREN: U1.13 (CHREN)
- new net GPIO4: J5.7 (Pin_7), U1.22 (GPIO.4)
- new net GPIO5: J5.8 (Pin_8), U1.21 (GPIO.5)
- new net GPIO6: U1.20 (GPIO.6)
- no-connect marks 1 -> 0
Other:
- note added: "ESP32 Reset Fix\nsee Voltlog #357"
- note added: "IO"
- note added: "USB to Serial Converter with auto-reset for ESP32 and ext LDO"
- note removed: "3.45V rail is capable of 100mA max!"
- note removed: "By default JP1 is closed and VIO = 3.45V"
- note removed: "USB to Serial Converter with auto-reset for ESP32"
- moved on the sheet: C2, C3, C4, C5, D2, D3, J1, J2, J4, J5, R4, R5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
