File: link.kicad_pcb (KiCad board)
At the start: 2 copper layers, 50 x 30 mm, 34 parts, among them J1 Link, J2 Standard, J3 USB_C_Receptacle_USB2.0, J4 Conn_01x08, J5 Conn_01x08, Q1 MMBT3904, Q2 MMBT3904, U1 CP2104

Commit message: Release revC
Parts:
- removed JP1: NC, Jumper:SolderJumper-2_P1.3mm_Open_TrianglePad1.0x1.5mm
- removed Q2: MMBT3904, Package_TO_SOT_SMD:SOT-23
- added C6: 1uF, Capacitor_SMD:C_0603_1608Metric, F.Cu at (143.1, 85.7)
- added U2: LR1107, Package_TO_SOT_SMD:SOT-89-3, F.Cu at (146.5, 97.5)
- C1: footprint Capacitor_SMD:C_0603_1608Metric -> Capacitor_SMD:C_1206_3216Metric
- D1: value SP0504BAHT -> SP0503BAHT; footprint Package_TO_SOT_SMD:SOT-23-5 -> Package_TO_SOT_SMD:SOT-143
- J3: footprint Voltlog:TYPE-C-31-M-12 -> voltlog:TYPE-C-31-M-12
- Q1: value MMBT3904 -> UMH3N; footprint Package_TO_SOT_SMD:SOT-23 -> Package_TO_SOT_SMD:SOT-363_SC-70-6
- R1: footprint Resistor_SMD:R_0603_1608Metric -> Resistor_SMD:R_1206_3216Metric
- R6: value 10K -> 1K
- R7: value 10K -> 22.1K
- R8: value 10K -> 47.5K
- U1: value CP2104 -> CP2102N-A01-GQFN28; footprint Package_DFN_QFN:QFN-24-1EP_4x4mm_P0.5mm_EP2.6x2.6mm -> Package_DFN_QFN:QFN-28-1EP_5x5mm_P0.5mm_EP3.35x3.35mm
- moved C2 23.9 mm to (143.0, 98.6), turned to -90 degrees
- moved C5 18.7 mm to (150.0, 98.6), turned to -90 degrees
- moved R7 16.1 mm to (124.5, 89.0)
- moved R8 16.1 mm to (124.5, 87.5), turned to 0 degrees
- moved D2 14.5 mm to (140.5, 79.0)
- moved D3 14.5 mm to (140.5, 93.5)
- moved R4 11.5 mm to (140.5, 80.5)
- moved R5 11.5 mm to (140.5, 92.0)
- moved Q1 3.81 mm to (140.3, 85.7), turned to 180 degrees
- moved R6 3.76 mm to (128.2, 90.8)
- moved R1 2.90 mm to (120.4, 77.6)
- moved C1 1.00 mm to (120.4, 80.0)
- moved D1 0.79 mm to (124.8, 83.2), turned to -90 degrees
- moved R3 0.25 mm to (120.5, 84.5)
- moved U1 0.25 mm to (133.0, 85.8)
Connections:
- net /EN renamed EN
- C2 pad 1: /VBUS -> VBUS
- C3 pad 1: /3.45V -> +3V3
- C4 pad 1: /3.45V -> +3V3
- C5 pad 1: Net-(C5-Pad1) -> +3V3
- D1 pad 1: /DM -> GND
- D1 pad 2: GND -> /USB_PWR
- D1 pad 4: /USB_PWR -> /DM
- D2 pad 2: /3.45V -> +3V3
- D3 pad 2: /3.45V -> +3V3
- F1 pad 1: /VBUS -> VBUS
- J1 pad 6: /3.45V -> +3V3
- J2 pad 6: /3.45V -> +3V3
- J4 pad 1: /VBUS -> VBUS
- J4 pad 2: /VIO -> /~{RST}
- J4 pad 3: GND -> /~{SUSPEND}
- J4 pad 4: /~RST -> /SUSPEND
- J4 pad 7: /3.45V -> +3V3
- J5 pad 7: /SUSPEND -> /GPIO4
- J5 pad 8: /~SUSPEND -> /GPIO5
- Q1 pad 1: Net-(Q1-Pad1) -> /DTR
- R4 pad 2: /GPIO1 -> /GPIO0
- R5 pad 2: /GPIO0 -> /GPIO1
- R6 pad 1: /~RST -> +3V3
- R6 pad 2: /VIO -> /~{RST}
- R7 pad 1: Net-(Q1-Pad1) -> VBUS
- R7 pad 2: /DTR -> Net-(R7-Pad2)
- R8 pad 1: Net-(Q2-Pad1) -> Net-(R7-Pad2)
- R8 pad 2: /RTS -> GND
- U1 pad 1: /RI -> /DCD
- U1 pad 11: /GPIO3 -> /~{SUSPEND}
- U1 pad 12: /GPIO2 -> /SUSPEND
- U1 pad 13: /GPIO1 -> /CHREN
- U1 pad 14: /GPIO0 -> /CHR1
- U1 pad 15: /~SUSPEND -> /CHR0
- U1 pad 16: Net-(C5-Pad1) -> /GPIO3
- U1 pad 17: /SUSPEND -> /GPIO2
- U1 pad 18: /CTS -> /GPIO1
- U1 pad 19: /RTS -> /GPIO0
- U1 pad 2: GND -> /RI
- U1 pad 20: /RXD -> /GPIO6
- U1 pad 21: /TXD -> /GPIO5
- U1 pad 22: /DSR -> /GPIO4
- U1 pad 23: /DTR -> /CTS
- U1 pad 24: /DCD -> /RTS
- U1 pad 25: GND -> /RXD
- U1 pad 3: /DP -> GND
- U1 pad 4: /DM -> /DP
- U1 pad 5: /VIO -> /DM
- U1 pad 6: /3.45V -> +3V3
- U1 pad 7: /VBUS -> +3V3
- U1 pad 8: /VBUS -> Net-(R7-Pad2)
- U1 pad 9: /~RST -> /~{RST}
Routing:
- net +3V3: track 0.00 -> 79.8 mm, vias 0 -> 2
- net /3.45V: track 75.2 -> 0.00 mm, vias 4 -> 0
- net VBUS: track 0.00 -> 39.3 mm, vias 0 -> 13
- net /VBUS: track 24.2 -> 0.00 mm
- net /VIO: track 22.1 -> 0.00 mm, vias 2 -> 0
- net /~RST: track 21.5 -> 0.00 mm
- net /~{RST}: track 0.00 -> 18.2 mm, vias 0 -> 1
- net /~SUSPEND: track 16.9 -> 0.00 mm, vias 2 -> 0
- net /~{SUSPEND}: track 0.00 -> 13.8 mm, vias 0 -> 1
- net /IO0: track 16.9 -> 30.2 mm, vias 0 -> 1
- net /GPIO5: track 0.00 -> 13.0 mm
- net Net-(R7-Pad2): track 0.00 -> 12.7 mm
- net /GPIO4: track 0.00 -> 11.4 mm
- net EN: track 23.0 -> 32.4 mm, vias 2 -> 1
- net Net-(Q2-Pad1): track 4.19 -> 0.00 mm
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- added copper zone on B.Cu, net VBUS
- added copper zone on F.Cu, net VBUS
Other:
- net class Default removed
- board text added: "3V3"
- board text added: "500mA max!"
- board text added: "IO2"
- board text added: "IO3"
- board text added: "IO4"
- board text added: "IO5"
- board text added: "revC"
- board text added: "~{RST}"
- board text added: "~{SUS}"
- board text removed: "100mA max!"
- board text removed: "3.4V"
- board text removed: "GPIO2"
- board text removed: "GPIO3"
- board text removed: "VIO"
- board text removed: "revA"
- board text removed: "~RST"
- board text removed: "~SUS"

Commit message: Release revE
Parts:
- removed the R4 at (140.5, 80.5)
- removed the R5 at (140.5, 92.0)
- removed R6: 1K, Resistor_SMD:R_0603_1608Metric
- added REF**: JLCPCB_tooling_hole, Voltlog:JLCPCB_tooling_hole, F.Cu at (119.2, 96.5)
- added REF**: JLCPCB_tooling_hole, Voltlog:JLCPCB_tooling_hole, F.Cu at (153.8, 72.5)
- added RN1: 1K, Resistor_SMD:R_Array_Convex_4x0603, F.Cu at (140.5, 87.5)
- added U2: USBLC6-2P6, Package_TO_SOT_SMD:SOT-666, F.Cu at (124.5, 85.2)
- added kibuzzard-623575FB: G***, kibuzzard-623575FB, F.Cu at (143.5, 92.5)
- added kibuzzard-6235760A: G***, kibuzzard-6235760A, F.Cu at (143.5, 79.5)
- added kibuzzard-62357631: G***, kibuzzard-62357631, F.Cu at (113.1, 92.5)
- added kibuzzard-623576E7: G***, kibuzzard-623576E7, F.Cu at (153.5, 82.1)
- added kibuzzard-623576F6: G***, kibuzzard-623576F6, F.Cu at (153.9, 79.6)
- added kibuzzard-62357705: G***, kibuzzard-62357705, F.Cu at (153.9, 84.8)
- added kibuzzard-62357716: G***, kibuzzard-62357716, F.Cu at (153.9, 87.3)
- added kibuzzard-62357727: G***, kibuzzard-62357727, F.Cu at (153.5, 89.9)
- added kibuzzard-62357731: G***, kibuzzard-62357731, F.Cu at (153.6, 92.5)
- added kibuzzard-62357776: G***, kibuzzard-62357776, F.Cu at (146.5, 94.2)
- added kibuzzard-623577BD: G***, kibuzzard-623577BD, F.Cu at (139.6, 95.6)
- added kibuzzard-623577CF: G***, kibuzzard-623577CF, F.Cu at (137.1, 95.6)
- added kibuzzard-623577DC: G***, kibuzzard-623577DC, F.Cu at (134.5, 95.6)
- added kibuzzard-623577E9: G***, kibuzzard-623577E9, F.Cu at (132.0, 95.6)
- added kibuzzard-623577F4: G***, kibuzzard-623577F4, F.Cu at (129.5, 95.6)
- added kibuzzard-62357894: G***, kibuzzard-62357894, F.Cu at (127.0, 95.3)
- added kibuzzard-623578AD: G***, kibuzzard-623578AD, F.Cu at (124.4, 95.3)
- added kibuzzard-623578BA: G***, kibuzzard-623578BA, F.Cu at (121.8, 95.1)
- added kibuzzard-623579BD: G***, kibuzzard-623579BD, F.Cu at (122.0, 75.3)
- added kibuzzard-623579CB: G***, kibuzzard-623579CB, F.Cu at (124.5, 76.3)
- added kibuzzard-623579D6: G***, kibuzzard-623579D6, F.Cu at (127.1, 76.3)
- added kibuzzard-623579E1: G***, kibuzzard-623579E1, F.Cu at (129.7, 76.3)
- added kibuzzard-623579ED: G***, kibuzzard-623579ED, F.Cu at (132.2, 76.3)
- added kibuzzard-623579F4: G***, kibuzzard-623579F4, F.Cu at (134.7, 76.3)
- added kibuzzard-623579FF: G***, kibuzzard-623579FF, F.Cu at (137.2, 76.3)
- added kibuzzard-62357A06: G***, kibuzzard-62357A06, F.Cu at (139.8, 76.3)
- added kibuzzard-62357A41: G***, kibuzzard-62357A41, B.Cu at (143.4, 86.1)
- added kibuzzard-62357A8A: G***, kibuzzard-62357A8A, B.Cu at (153.9, 79.6)
- added kibuzzard-62357AC8: G***, kibuzzard-62357AC8, B.Cu at (153.5, 82.1)
- added kibuzzard-62357AF5: G***, kibuzzard-62357AF5, B.Cu at (153.9, 84.8)
- added kibuzzard-62357B09: G***, kibuzzard-62357B09, B.Cu at (153.9, 87.3)
- added kibuzzard-62357B18: G***, kibuzzard-62357B18, B.Cu at (153.5, 89.9)
- added kibuzzard-62357B23: G***, kibuzzard-62357B23, B.Cu at (153.6, 92.5)
- added kibuzzard-62357B61: G***, kibuzzard-62357B61, B.Cu at (139.6, 95.6)
- added kibuzzard-62357B6B: G***, kibuzzard-62357B6B, B.Cu at (137.1, 95.6)
- added kibuzzard-62357B85: G***, kibuzzard-62357B85, B.Cu at (134.5, 95.6)
- added kibuzzard-62357B8F: G***, kibuzzard-62357B8F, B.Cu at (132.0, 95.6)
- added kibuzzard-62357B96: G***, kibuzzard-62357B96, B.Cu at (129.5, 95.6)
- added kibuzzard-62357B9D: G***, kibuzzard-62357B9D, B.Cu at (127.0, 95.3)
- added kibuzzard-62357BA3: G***, kibuzzard-62357BA3, B.Cu at (124.4, 95.3)
- added kibuzzard-62357BA9: G***, kibuzzard-62357BA9, B.Cu at (121.8, 95.1)
- added kibuzzard-62357BE4: G***, kibuzzard-62357BE4, B.Cu at (139.8, 76.3)
- added kibuzzard-62357BED: G***, kibuzzard-62357BED, B.Cu at (137.2, 76.3)
- added kibuzzard-62357BF2: G***, kibuzzard-62357BF2, B.Cu at (134.7, 76.3)
- added kibuzzard-62357BF8: G***, kibuzzard-62357BF8, B.Cu at (132.2, 76.3)
- added kibuzzard-62357BFE: G***, kibuzzard-62357BFE, B.Cu at (129.7, 76.3)
- added kibuzzard-62357C0A: G***, kibuzzard-62357C0A, B.Cu at (127.1, 76.3)
- added kibuzzard-62357C11: G***, kibuzzard-62357C11, B.Cu at (124.5, 76.3)
- added kibuzzard-62357C18: G***, kibuzzard-62357C18, B.Cu at (122.0, 75.8)
- C3: renamed from C5; value 4.7uF -> 10uF
- C5: renamed from C3; value 4.7uF -> 10uF
- D1: value SP0503BAHT -> PWR; footprint Package_TO_SOT_SMD:SOT-143 -> LED_SMD:LED_0603_1608Metric
- moved D1 12.4 mm to (116.5, 92.5), turned to 0 degrees
- moved C4 5.15 mm to (140.5, 81.2), turned to 180 degrees
- moved Q1 1.96 mm to (140.5, 83.8)
- moved D3 1.00 mm to (140.5, 92.5)
- moved D2 0.50 mm to (140.5, 79.5)
- moved FID1 0.46 mm to (112.0, 94.2)
- moved R3 0.25 mm to (120.5, 84.2)
- renumbered C6 to C4, C4 to C6, R7 to R4, R8 to R5, U2 to U1, U1 to U3
Connections:
- D1 pad 2: /USB_PWR -> Net-(D1-Pad2)
- J3 pad A8: Net-(J3-PadA8) -> unconnected-(J3-PadA8)
- J3 pad B8: Net-(J3-PadB8) -> unconnected-(J3-PadB8)
- U3 pad 10: Net-(U1-Pad10) -> unconnected-(U3-Pad10)
- U3 pad 4: /DP -> Net-(U2-Pad6)
- U3 pad 5: /DM -> Net-(U2-Pad4)
Routing:
- net Net-(D1-Pad2): track 0.00 -> 25.8 mm, vias 0 -> 4
- net /DM: track 26.1 -> 11.2 mm
- net Net-(D3-Pad1): track 1.50 -> 13.7 mm
- net /~{RST}: track 18.2 -> 27.1 mm, vias 1 -> 3
- net /DP: track 17.7 -> 9.47 mm
- net Net-(D2-Pad1): track 1.50 -> 9.12 mm
- net Net-(U2-Pad6): track 0.00 -> 5.63 mm
- net Net-(U2-Pad4): track 0.00 -> 5.39 mm
- net /GPIO0: track 8.57 -> 4.58 mm
- net /GPIO1: track 8.48 -> 4.71 mm
- net Net-(R4-Pad2): track 12.7 -> 10.0 mm
- net /USB_PWR: track 7.16 -> 9.68 mm
- net EN: track 32.4 -> 30.5 mm
- net /IO0: track 30.2 -> 28.7 mm
- net /DTR: track 27.3 -> 25.9 mm
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Other:
- board text added: "revE"
- board text removed: "500mA max!"
- board text removed: "CTS"
- board text removed: "DCD"
- board text removed: "DSR"
- board text removed: "DTR"
- board text removed: "G"
- board text removed: "IO2"
- board text removed: "IO3"
- board text removed: "IO4"
- board text removed: "IO5"
- board text removed: "RI"
- board text removed: "RTS"
- board text removed: "RX"
- board text removed: "SUS"
- board text removed: "TX"
- board text removed: "VBUS"
- board text removed: "WWW.VOLTLOG.COM"
- board text removed: "revC"
- board text removed: "~{RST}"
- board text removed: "~{SUS}"

Commit message: revE release
Parts:
- removed FID1, FID2, FID3: Fiducial, Fiducial:Fiducial_0.5mm_Mask1mm
- removed REF** (x2): JLCPCB_tooling_hole, Voltlog:JLCPCB_tooling_hole
- J3: footprint voltlog:TYPE-C-31-M-12 -> Voltlog:TYPE-C-31-M-12
Other:
- board text added: "1723"
