File: link.kicad_sch (KiCad schematic)
At the start: 34 parts, among them J1 Link, J2 Standard, J3 USB_C_Receptacle_USB2.0, J4 Conn_01x08, J5 Conn_01x08, Q1 UMH3N, U1 CP2102N-A01-GQFN28, U2 LR1107

Commit message: Release revE
Parts:
- removed D1: SP0503BAHT, Package_TO_SOT_SMD:SOT-143, symbol Power_Protection:SP0503BAHT
- removed R4, R5, R6: 1K, Resistor_SMD:R_0603_1608Metric, symbol Device:R_US
- added D1: PWR, LED_SMD:LED_0603_1608Metric, symbol Device:LED_ALT
- added RN1: 1K, Resistor_SMD:R_Array_Convex_4x0603, symbol Device:R_Pack04_Split
- added U2: USBLC6-2P6, Package_TO_SOT_SMD:SOT-666, symbol Power_Protection:USBLC6-2P6
- C1: LCSC (none) -> C107198; PN (none) -> CC1206KKX7RCBB472; Voltage (none) -> 1KV
- C2: LCSC (none) -> C1592; PN (none) -> CL10A105KO8NNNC
- C3: renamed from C5; value 4.7uF -> 10uF; LCSC (none) -> C92487; PN (none) -> CL10A106MO8NQNC; Voltage (none) -> 16V
- C5: renamed from C3; value 4.7uF -> 10uF
- C6: renamed from C4; LCSC (none) -> C24452; PN (none) -> CL10B104JB8NNNC
- D2: LCSC (none) -> C84267; PN (none) -> NCD0603G1
- D3: LCSC (none) -> C193902; PN (none) -> NCD0603R5
- F1: LCSC (none) -> C207014; PN (none) -> 0603L050SLYR
- J1: LCSC (none) -> C145963; PN (none) -> BOOMELE
- J3: LCSC (none) -> C165948; PN (none) -> TYPE-C-31-M-12
- Q1: LCSC (none) -> C62892; PN (none) -> UMH3N
- U1: renamed from U2; LCSC (none) -> C171498; PN (none) -> LR1107G-33-AB3-C-R
- U3: renamed from U1; LCSC (none) -> C964632; PN (none) -> CP2102N-A02-GQFN28R
- renumbered C6 to C4, R7 to R4, R8 to R5
Connections:
- net +3V3: now also RN1.5 (R4.2), RN1.6 (R3.2)
- net DM: now also U2.3 (I/O2); no longer U3.5 (D-)
- net DP: now also U2.1 (I/O1); no longer U3.4 (D+)
- net GND: now also D1.1 (K), U2.2 (GND)
- net GPIO0: now also RN1.1 (R1.1)
- net GPIO1: now also RN1.2 (R2.1)
- net USB_PWR: now also U2.5 (VBUS)
- net ~{RST}: now also RN1.3 (R3.1)
- net at D2.1 (K): now also RN1.8 (R1.2)
- net at D3.1 (K): now also RN1.7 (R2.2)
- new net: U2.6 (I/O1), U3.4 (D+)
- new net: U2.4 (I/O2), U3.5 (D-)
- new net: D1.2 (A), RN1.4 (R4.1)
Other:
- moved on the sheet: C2, C3, F1, U1

Commit message: revE release
Parts:
- removed FID1, FID2, FID3: Fiducial, Fiducial:Fiducial_0.5mm_Mask1mm, symbol Mechanical:Fiducial
- C2: LCSC C1592 -> C15849
- C3: LCSC C92487 -> C19702
- C4: LCSC (none) -> C15849
- C5: LCSC (none) -> C19702
- C6: LCSC C24452 -> C14663
- J3: footprint voltlog:TYPE-C-31-M-12 -> Voltlog:TYPE-C-31-M-12
- R4: LCSC (none) -> C25961
- R5: LCSC (none) -> C203634
- RN1: LCSC (none) -> C20197; PN (none) -> 4D03WGF1001T5E
- RN1: LCSC C425239 -> C20197
- U2: LCSC (none) -> C2827693
- U3: LCSC C964632 -> C1550553
